File: Hardware/FluxSens_V2/FluxSens_V2.kicad_sch (KiCad schematic)
At the start: 35 parts, among them J1 Conn_01x08, U1 HMC1051Z, U2 RC4558, U3 MAX662ACSA+

Commit message: finished the V2 board layout
Parts:
- removed C1, C12, C8: 100nf, Capacitor_SMD:C_0805_2012Metric_Pad1.18x1.45mm_HandSolder, symbol Device:C_Small
- removed C10, C3, C7: C_Polarized_Small, Capacitor_Tantalum_SMD:CP_EIA-7343-31_Kemet-D_Pad2.25x2.55mm_HandSolder, symbol Device:C_Polarized_Small
- removed C9: 2uf, Capacitor_SMD:C_0805_2012Metric_Pad1.18x1.45mm_HandSolder, symbol Device:C_Small
- added 12V1, 20V1, 5V1, J_+Vbias1, J_-Vbias1, S/R1, S/R_PWR1, Vcc1, Vout1: Conn_01x02, Connector_PinHeader_2.54mm:PinHeader_1x02_P2.54mm_Horizontal, symbol Connector_Generic:Conn_01x02
- added C10, C13, C14: 100nf, Capacitor_SMD:C_0805_2012Metric_Pad1.18x1.45mm_HandSolder, symbol Device:C_Small
- added C12, C8, C9: C_Polarized_Small, Capacitor_Tantalum_SMD:CP_EIA-7343-31_Kemet-D_Pad2.25x2.55mm_HandSolder, symbol Device:C_Polarized_Small
- added C3: 1u, Capacitor_SMD:C_0805_2012Metric_Pad1.18x1.45mm_HandSolder, symbol Device:C_Small
- added C7: C_Small, Capacitor_SMD:C_0805_2012Metric_Pad1.18x1.45mm_HandSolder, symbol Device:C_Small
- added H1, H2: MountingHole, MountingHole:MountingHole_3.2mm_M3, symbol Mechanical:MountingHole
- added Q1: BSD235C, Package_TO_SOT_SMD:SOT-563, symbol Transistor_FET:BSD235C
- added R19: Rth, Resistor_SMD:R_0805_2012Metric_Pad1.20x1.40mm_HandSolder, symbol Device:R_Small
- added R20: 4k7, Resistor_SMD:R_0805_2012Metric_Pad1.20x1.40mm_HandSolder, symbol Device:R_Small
- added R21: 180R, Resistor_SMD:R_0805_2012Metric_Pad1.20x1.40mm_HandSolder, symbol Device:R_Small
- added R22, R24: 0R, Resistor_SMD:R_0805_2012Metric_Pad1.20x1.40mm_HandSolder, symbol Device:R_Small
- added R23: 10k, Resistor_SMD:R_0805_2012Metric_Pad1.20x1.40mm_HandSolder, symbol Device:R_Small
- added TP_12V1, TP_20V1, TP_5V1, TP_GND1, TP_GND2, TP_GND3, TP_S/R-PWR1, TP_S/R1, TP_Vbias+1, TP_Vbias-1, TP_Vcc/2, TP_Vcc1, TP_Vo+1, TP_Vo-1, TP_Vout1, TP_Vout_mid1: TestPoint, TestPoint:TestPoint_THTPad_D2.5mm_Drill1.2mm, symbol Connector:TestPoint
- C11: value 100nf -> 2uf
- C2: value C_Small -> 1u
- C5: value C_Small -> 100nf
- R1: value R_Small -> 10k
- R12, R5: value 500k -> R_Small
- R13: value Rb -> 4R
- R14: value R_Small -> 4R
- R15: value Ra -> 500k
- R16: value Rth -> Rb
- R17: value R_Small -> Ra
- R6: value 5k -> 500k
- R8: value R_Small -> 5k
- U1: now left out of the parts list
Connections:
- net S/R- is gone; now on net -Vbias: R4.2
- net +12V: now also D1.2 (A), U3.6 (VOUT), 12V1.1 (Pin_1), C10.2, TP_12V1.1
- net 20V: now also 20V1.1 (Pin_1), C14.2, TP_20V1.1
- net GND: now also C2.1, C4.1, R16.1, R5.2, C3.1, C8.2, J_+Vbias1.2 (Pin_2), J_-Vbias1.2 (Pin_2), Q1.1 (SN), R20.1, R23.1, S/R1.2 (Pin_2), S/R_PWR1.2 (Pin_2), TP_GND1.1, TP_GND3.1, Vcc1.2 (Pin_2), Vout1.2 (Pin_2); no longer C5.1, R1.2, R13.1, R3.2, R9.2, U3.7 (GND), U3.8 (SHDN)
- net S/R+: now also R11.2, C7.1; no longer R10.2
- net Vcc: now also C4.2, R1.2, TP_Vcc1.1, Vcc1.1 (Pin_1); no longer C5.2, R14.1, R2.2
- net Vcc/2: now also R1.1, R6.1, R23.2, TP_Vcc/2.1; no longer R5.1
- net Vo: now also R17.2, R19.2, TP_Vout1.1, Vout1.1 (Pin_1); no longer R15.2, R16.2
- net Vo+: now also R7.1, R9.2, TP_Vo+1.1; no longer R6.1, R8.2
- net Vo-: now also R12.2, R8.1, TP_Vo-1.1; no longer R11.2, R7.1
- net at R14.2: now also J_+Vbias1.1 (Pin_1)
- net at R4.1: now also J1.5 (Pin_5); no longer J1.7 (Pin_7)
- net at R6.2, U2.3 (+): now also R7.2; no longer R5.2
- net at U3.1 (C1-): now also C9.2
- net at U3.2 (C1+): now also C9.1
- net at U3.3 (C2-): now also C12.2, C13.2; no longer C11.2
- net at U3.4 (C2+): now also C12.1
- net at D1.1 (K), D2.2 (A): now also C13.1; no longer C11.1
- net at U2.1, U2.5 (+): now also C5.2, R15.2, TP_Vout_mid1.1; no longer R12.2
- net at J1.1 (Pin_1): now also R2.1; no longer R1.1
- net at J1.2 (Pin_2): now also R9.1; no longer R8.1
- net at J1.3 (Pin_3): now also R3.1; no longer R2.1
- net at J1.4 (Pin_4): now also R10.1; no longer R9.1
- net at J1.6 (Pin_6): now also R11.1; no longer R10.1
- net at J1.8 (Pin_8): now also R12.1; no longer R11.1
- net -Vbias: now reaches C2.2
- net -Vbias: now also R10.2, R13.1, R2.2, TP_Vbias-1.1
- net at R17.1: now also R16.2, U2.6 (-), R19.1
- net +5V renamed 5V
- net 5V: now also C11.2, 5V1.1 (Pin_1), TP_5V1.1
- new net: C7.2, Q1.3 (DP), Q1.6 (DN)
- new net: J1.7 (Pin_7), R5.1
- new net: C8.1, R21.2, R22.2
- new net: J_-Vbias1.1 (Pin_1), R13.2
- new net: R21.1, S/R_PWR1.1 (Pin_1), TP_S/R-PWR1.1
- new net: C5.1, R15.1, R8.2, U2.2 (-)
- new net: Q1.4 (SP), R22.1
- new net: R24.2, S/R1.1 (Pin_1), TP_S/R1.1
- new net +Vbias: C3.2, R14.1, R3.2, TP_Vbias+1.1
- new net GND2: 12V1.2 (Pin_2), 20V1.2 (Pin_2), 5V1.2 (Pin_2), C10.1, C11.1, C14.1, TP_GND2.1, U3.7 (GND), U3.8 (SHDN)
- new net S/R: Q1.2 (GN), Q1.5 (GP), R20.2, R24.1

Commit message: update
Parts:
- C10, C13, C14, C5: value 100nf -> 100nF
- C11: value 2uf -> 2u
- C12, C8, C9: value C_Polarized_Small -> 4.7u
- C2, C3: value 1u -> 1uF
- C4: value C_Small -> 1uF
- C6, C7: value C_Small -> 0.1uF
- R10, R11, R12, R2, R3, R4, R5, R9: value R_Small -> 0R
- R13, R14: value 4R -> 3R9
- R15, R6: value 500k -> 510k
- R16: value Rb -> 51k
- R17/C17: renamed from R17; value Ra -> 82nF
- R19: value Rth -> 51k
- R7, R8: value 5k -> 5k1
Other:
- note added: "1."
- note added: "2."
- note added: "Nobīdes spriegums sensoram"
- note added: "OP Barošanas sprieguma ķēde"
- note added: "OP Ķēde"
- note added: "REF priekš OP Ķēdes"
- note added: "S/R Barošanas ķēde"
- note added: "Sensora pieslēguma ķēde"
- moved on the sheet: 12V1, 20V1, 5V1, C10, C11, C12, C13, C14, C2, C3, C4, C5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
